Commit message: collision change for grasp

File: mani_skill/agents/robots/SO100/urdf/SO100.urdf (robot description, URDF)
Before this commit: robot SO100, 7 links, 6 joints
Links:
- link Fixed_Jaw: geometry collision box size=0.12 0.02 0.03; visual mesh filename=package://SO100/meshes/Fixed_Jaw.STL

Commit message: add hhr.glb to the env;FPS control;urdf change

File: mani_skill/agents/robots/SO100/urdf/SO100.urdf (robot description, URDF)
Before this commit: robot SO100, 7 links, 6 joints
Links:
- link Fixed_Jaw: geometry collision box size=0.1 0.02 0.03; visual mesh filename=package://SO100/meshes/Fixed_Jaw.STL
